Commit message: Minor Changes

File: urdf/robot.urdf (robot description, URDF)
Before this commit: robot Gundum, 34 links, 33 joints
Links:
- removed link left_shoulder_link
- removed link right_shoulder_link
Joints:
- removed joint left_arm_shoulder
- removed joint right_arm_shoulder
- added joint left_leg_joint: type fixed, parent left_feet_link, child left_feet, origin xyz=.1 0 -.25 rpy=0 0 0
- added joint right_leg_joint: type fixed, parent right_feet_link, child right_feet, origin xyz=.1 0 -.25 rpy=0 0 0
- joint left_elbow_joint: limit lower=-3.146 upper=3.146 effort=10 velocity=3 -> lower=-1.55 upper=1.55 effort=10 velocity=3
- joint left_hand_joint: child left_feet -> left_hand_link; origin xyz=.1 0 -.25 rpy=0 0 0 -> xyz=0 0 -.55 rpy=0 0 0; parent left_feet_link -> left_wrist_link
- joint left_shoulder_forward_joint: parent left_shoulder_link -> shoulder_link
- joint neck_shoulder_link_joint: limit lower=-3.146 upper=3.146 effort=10 velocity=3 -> lower=-1.55 upper=1.55 effort=10 velocity=3
- joint right_elbow_joint: limit lower=-3.146 upper=3.146 effort=10 velocity=3 -> lower=-1.5 upper=1.5 effort=10 velocity=3
- joint right_hand_joint: child right_feet -> right_hand_link; origin xyz=.1 0 -.25 rpy=0 0 0 -> xyz=0 0 -.55 rpy=0 0 0; parent right_feet_link -> right_wrist_link
- joint right_shoulder_forward_joint: parent right_shoulder_link -> shoulder_link

Commit message: Add files via upload

File: urdf/robot.urdf (robot description, URDF)
Before this commit: robot Gundum, 32 links, 33 joints
Links:
- link head_link: mass None -> 0.18; geometry collision box size=0.9 0.9 .9; visual box size=0.9 0.9 .9
- link hip_link: mass None -> 0.18; geometry collision box size=0.25 0.5 3; visual box size=0.25 0.5 3
- link left_elbow_link: mass None -> 0.18; geometry collision box size=0.35 0.35 .5; visual box size=0.35 0.35 .5
- link left_feet: mass None -> 0.18; geometry collision box size=.6 .4 .1; visual box size=.6 .4 .1
- link left_feet_link: mass None -> 0.18; geometry collision box size=.3 .5 .3; visual box size=.3 .5 .3
- link left_hand_link: mass None -> 0.18; geometry collision box size=0.3 0.1 0.6; visual box size=0.3 0.1 0.6
- link left_hip_forward_link: mass None -> 0.18; geometry collision box size=.3 .5 .3; visual box size=.3 .5 .3
- link left_hip_up_link: mass None -> 0.18; geometry collision box size=.3 .5 .3; visual box size=.3 .5 .3
- link left_knee_link: mass None -> 0.18; geometry collision box size=.35 0.35 .5; visual box size=.35 0.35 .5
- link left_lower_arm_link: mass None -> 0.18; geometry collision cylinder length=1.1 radius=0.075; visual cylinder length=1.1 radius=0.075
- link left_lower_leg_link: mass None -> 0.18; geometry collision cylinder length=1.1 radius=0.075; visual cylinder length=1.1 radius=0.075
- link left_shoulder_forward_link: mass None -> 0.18; geometry collision box size=0.3 0.5 0.3; visual box size=0.3 0.5 0.3
- link left_shoulder_up_link: mass None -> 0.18; geometry collision box size=0.3 0.5 0.3; visual box size=0.3 0.5 0.3
- link left_upper_arm_link: mass None -> 0.18; geometry collision cylinder length=0.5 radius=0.075; visual cylinder length=0.5 radius=0.075
- link left_upper_leg_link: mass None -> 0.18; geometry collision cylinder length=.5 radius=0.075; visual cylinder length=.5 radius=0.075
- link left_wrist_link: mass None -> 0.18; geometry collision box size=0.3 0.5 0.3; visual box size=0.3 0.5 0.3
- link neck_link: mass None -> 0.18; geometry collision box size=0.25 0.30 .5; visual box size=0.25 0.30 .5
- link right_elbow_link: mass None -> 0.18; geometry collision box size=0.35 0.35 .5; visual box size=0.35 0.35 .5
- link right_feet: mass None -> 0.18; geometry collision box size=.6 .4 .1; visual box size=.6 .4 .1
- link right_feet_link: mass None -> 0.18; geometry collision box size=.3 .5 .3; visual box size=.3 .5 .3
- link right_hand_link: mass None -> 0.18; geometry collision box size=.3 .1 .6; visual box size=.3 .1 .6
- link right_hip_forward_link: mass None -> 0.18; geometry collision box size=.3 .5 .3; visual box size=.3 .5 .3
- link right_hip_up_link: mass None -> 0.18; geometry collision box size=.3 .5 .3; visual box size=.3 .5 .3
- link right_knee_link: mass None -> 0.18; geometry collision box size=.35 .35 .5; visual box size=.35 .35 .5
- link right_lower_arm_link: mass None -> 0.18; geometry collision cylinder length=1.1 radius=0.075; visual cylinder length=1.1 radius=0.075
- link right_lower_leg_link: mass None -> 0.18; geometry collision cylinder length=1.1 radius=0.075; visual cylinder length=1.1 radius=0.075
- link right_shoulder_forward_link: mass None -> 0.18; geometry collision box size=0.3 0.5 0.3; visual box size=0.3 0.5 0.3
- link right_shoulder_up_link: mass None -> 0.18; geometry collision box size=0.3 0.5 0.3; visual box size=0.3 0.5 0.3
- link right_upper_arm_link: mass None -> 0.18; geometry collision cylinder length=.5 radius=0.075; visual cylinder length=.5 radius=0.075
- link right_upper_leg_link: mass None -> 0.18; geometry collision cylinder length=.5 radius=0.075; visual cylinder length=.5 radius=0.075
- link right_wrist_link: mass None -> 0.18; geometry collision box size=.3 .5 .3; visual box size=.3 .5 .3
- link shoulder_link: mass None -> 0.18; geometry collision box size=0.3 2.4 0.5; visual box size=0.3 2.4 0.5
